Commit message: add missing prefix on joint5b for irb5400

File: abb_irb5400_support/urdf/irb5400_macro.xacro (robot description, xacro)
@@ -160,5 +160,5 @@
         <axis xyz="1 0 0"/>
         <limit lower="-6.0" upper="6.0" effort="100" velocity="6.1086"/>
-        <mimic joint="joint_5" multiplier="-1.0" offset="0"/>
+	<mimic joint="${prefix}joint_5" multiplier="-1.0" offset="0"/>
     </joint>
     <joint name="${prefix}joint_6" type="revolute">
